Commit message: attempt at speeding up the robot, did not work yield any improvements

File: simulation_ws/src/warehouse_simulation/urdf/robot.urdf (robot description, URDF)
Before this commit: robot warehouse_robot, 4 links, 3 joints
Links:
- link base_link: mass 20.0 -> 5.0
- link left_wheel: mass 0.2 -> 0.5
- link right_wheel: mass 0.2 -> 0.5
